File: 03_Projekt/02_TinkerCAD/IG1_LEDProjekt.brd (EAGLE design)
At the start: 68.6 x 53.3 mm, 17 parts, among them P1 5V

Commit message: Structorizer /Thinker CAD
Parts:
- removed P1: 5V, AUTODESK_CIRCUITS_BREADBOARD:2P-2.54-65/35MIL
- removed Rpot1: 250k‎Ω, AUTODESK_CIRCUITS_BREADBOARD:B25V
- removed U1: (no value), AUTODESK_CIRCUITS_BREADBOARD:TO92
- added D7: BLUE, Tinkercad:LEDRD254W60D565H860B_B
- added DIST1: DISTANCE-SENSOR-4PINHC-SR04, Tinkercad:HC-SR04
- added R7: 470, Tinkercad:RESAD1016W63L850D250B
- D1, D2: value (none) -> GREEN; device AUTODESK_CIRCUITS_BREADBOARD:LED5MM -> Tinkercad:LEDRD254W60D565H860B_G
- D3, D4: value (none) -> YELLOW; device AUTODESK_CIRCUITS_BREADBOARD:LED5MM -> Tinkercad:LEDRD254W60D565H860B_Y
- D5, D6: value (none) -> RED; device AUTODESK_CIRCUITS_BREADBOARD:LED5MM -> Tinkercad:LEDRD254W60D565H860B
- R1, R2, R3, R4, R5, R6: value 200‎Ω -> 470; device AUTODESK_CIRCUITS_BREADBOARD:0207/10 -> Tinkercad:RESAD1016W63L850D250B
- S1: value (none) -> SWITCH_MOMENTARY; device AUTODESK_CIRCUITS_BREADBOARD:TL1105 -> Tinkercad:SWITCH-MOMENTARY-PTH-6.5MM
- U2: value (none) -> ARDUINO-UNO-R3-SHIELD; device AUTODESK_CIRCUITS_BREADBOARD:ARDUINO_UNO -> Tinkercad:ARDUINO-UNO-R3-SHIELD
- moved S1 130.9 mm to (70.8, 123.2), turned to 90 degrees
- moved D1 109.5 mm to (11.1, 132.1), turned to 180 degrees
- moved D2 97.3 mm to (16.2, 132.1), turned to 180 degrees
- moved R6 97.0 mm to (37.8, 122.0), turned to 90 degrees
- moved D3 85.5 mm to (21.3, 132.1), turned to 180 degrees
- moved R5 83.3 mm to (32.7, 122.0), turned to 90 degrees
- moved U2 75.6 mm to (45.6, 47.9)
- moved D4 74.4 mm to (26.4, 132.1), turned to 180 degrees
- moved R4 69.7 mm to (27.6, 122.0), turned to 90 degrees
- moved D5 64.3 mm to (31.5, 132.1), turned to 180 degrees
- moved R3 56.0 mm to (22.6, 122.0), turned to 90 degrees
- moved D6 55.7 mm to (36.5, 132.1), turned to 180 degrees
- moved R2 42.4 mm to (17.5, 122.0), turned to 90 degrees
- moved R1 28.8 mm to (12.4, 122.0), turned to 90 degrees
Connections:
- removed net N$1: S1.1, U1.3, U2.7
- removed net N$10: R3.1, U2.11
- removed net N$11: R4.1, U2.10
- removed net N$12: R5.1, U2.9
- removed net N$13: R6.1, U2.8
- removed net N$2: S1.3, U2.6
- removed net N$3: D1.A, D2.A, D3.A, D4.A, D5.A, D6.A, P1.2, R1.2, R2.2, R3.2, R4.2, R5.2, R6.2
- removed net N$4: U1.2
- removed net N$5: D1.K, D2.K, D3.K, D4.K, D5.K, D6.K, P1.1, Rpot1.E, S1.2, S1.4, U1.1, U2.GND
- removed net N$6: Rpot1.A, U2.5
- removed net N$7: Rpot1.S
- removed net N$8: R1.1, U2.13
- removed net N$9: R2.1, U2.12
- new net U2_5V: D1.1, D2.1, D3.1, D4.1, D5.1, D6.1, D7.1, DIST1.1, R1.2, R2.2, R3.2, R4.2, R5.2, R6.2, R7.2, U2.5V
- new net U2_A0: DIST1.2, U2.A0
- new net U2_A1: R7.1, U2.A1
- new net U2_D2: R3.1, U2.D2
- new net U2_D3: R4.1, U2.D3
- new net U2_D4: R5.1, U2.D4
- new net U2_D5: R6.1, U2.D5
- new net U2_D8: S1.3, S1.4, U2.D8
- new net U2_GND: D1.2, D2.2, D3.2, D4.2, D5.2, D6.2, D7.2, DIST1.3, S1.1, S1.2, U2.GND@0, U2.GND@1, U2.GND@2
- new net U2_RX: R1.1, U2.RX
- new net U2_TX: R2.1, U2.TX
Other:
- board size 68.6 x 53.3 mm -> 88 x 144.8 mm
